Commit message: Reduced the weight of the VI sensor to avoid changing controller parameters. This is a hack and needs to be solved properly.

File: rotors_description/urdf/component_snippets.xacro (robot description, xacro)
@@ -519,5 +519,6 @@
       </visual>
       <inertial>
-        <mass value="0.13" />
+        <!--mass value="0.13" /-->
+        <mass value="1e-6" />
         <origin xyz="0 0 0" rpy="0 0 0" />
         <inertia ixx="1e-6" ixy="0" ixz="0" iyy="1e-6" iyz="0" izz="1e-6" />
